Commit message: Add t800 support

File: assets/resource/robot/pm01_edu/urdf/serial_pm01_edu.urdf (robot description, URDF)
Before this commit: robot engineai_pm01, 29 links, 28 joints
Links:
- link LINK_BASE: geometry collision sphere radius=0.0725; visual mesh filename=package://resource/robot/pm01_edu/meshes/LINK_BASE.dae
- link LINK_ELBOW_END_L: geometry collision sphere radius=0.05
- link LINK_ELBOW_END_R: geometry collision sphere radius=0.05
- link LINK_ELBOW_YAW_L: geometry collision cylinder length=0.07 radius=0.03; visual mesh filename=package://resource/robot/pm01_edu/meshes/LINK_ELBOW_YAW_L.d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
- link LINK_ELBOW_YAW_R: geometry collision cylinder length=0.07 radius=0.03; visual mesh filename=package://resource/robot/pm01_edu/meshes/LINK_ELBOW_YAW_R.d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
- link LINK_HEAD_YAW: geometry collision sphere radius=0.1; visual mesh filename=package://resource/robot/pm01_edu/meshes/LINK_HEAD_YAW.dae
- link LINK_HIP_PITCH_L: geometry collision cylinder length=0.10 radius=0.048; visual mesh filename=package://resource/robot/pm01_edu/meshes/LINK_HIP_PITCH_L.d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
- link LINK_HIP_PITCH_R: geometry collision cylinder length=0.10 radius=0.048; visual mesh filename=package://resource/robot/pm01_edu/meshes/LINK_HIP_PITCH_R.d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
- link LINK_HIP_ROLL_L: geometry collision cylinder length=0.02 radius=0.06; visual mesh filename=package://resource/robot/pm01_edu/meshes/LINK_HIP_ROLL_L.dae
- link LINK_HIP_ROLL_R: geometry collision cylinder length=0.02 radius=0.06; visual mesh filename=package://resource/robot/pm01_edu/meshes/LINK_HIP_ROLL_R.dae
- link LINK_HIP_YAW_L: geometry collision cylinder length=0.02 radius=0.05; collision cylinder length=0.02 radius=0.05
- link LINK_HIP_YAW_R: geometry collision cylinder length=0.02 radius=0.05; collision cylinder length=0.02 radius=0.05
- link LINK_TORSO_YAW: geometry collision box size=0.15 0.17 0.08; collision box size=0.18 0.2 0.2
Joints:
- joint J02_HIP_YAW_L: limit lower=-1.57 upper=4.014 effort=50 velocity=35.2 -> lower=-1.57 upper=4.014 effort=61 velocity=35.2
- joint J04_ANKLE_PITCH_L: limit lower=-0.6807 upper=0.7243 effort=50 velocity=35.2 -> lower=-0.6807 upper=0.7243 effort=61 velocity=35.2
- joint J05_ANKLE_ROLL_L: limit lower=-0.2618 upper=0.2618 effort=50 velocity=35.2 -> lower=-0.2618 upper=0.2618 effort=61 velocity=35.2
- joint J08_HIP_YAW_R: limit lower=-4.014 upper=1.57 effort=50 velocity=35.2 -> lower=-4.014 upper=1.57 effort=61 velocity=35.2
- joint J10_ANKLE_PITCH_R: limit lower=-0.6807 upper=0.7243 effort=50 velocity=35.2 -> lower=-0.6807 upper=0.7243 effort=61 velocity=35.2
- joint J11_ANKLE_ROLL_R: limit lower=-0.2618 upper=0.2618 effort=50 velocity=35.2 -> lower=-0.2618 upper=0.2618 effort=61 velocity=35.2
- joint J12_WAIST_YAW: limit lower=-4.014 upper=1.57 effort=50 velocity=35.2 -> lower=-4.014 upper=1.57 effort=61 velocity=35.2
- joint J13_SHOULDER_PITCH_L: limit lower=-2.9671 upper=2.7925 effort=50 velocity=35.2 -> lower=-2.9671 upper=2.7925 effort=61 velocity=35.2
- joint J14_SHOULDER_ROLL_L: limit lower=-0.6108 upper=2.3562 effort=50 velocity=35.2 -> lower=-0.6108 upper=2.3562 effort=61 velocity=35.2
- joint J15_SHOULDER_YAW_L: limit lower=-2.618 upper=2.618 effort=50 velocity=35.2 -> lower=-2.618 upper=2.618 effort=61 velocity=35.2
- joint J16_ELBOW_PITCH_L: limit lower=-2.1948 upper=0.7374 effort=50 velocity=35.2 -> lower=-2.1948 upper=0.7374 effort=61 velocity=35.2
- joint J17_ELBOW_YAW_L: limit lower=-2.618 upper=2.618 effort=50 velocity=35.2 -> lower=-2.618 upper=2.618 effort=61 velocity=35.2
- joint J18_SHOULDER_PITCH_R: limit lower=-2.9671 upper=2.7925 effort=50 velocity=35.2 -> lower=-2.9671 upper=2.7925 effort=61 velocity=35.2
- joint J19_SHOULDER_ROLL_R: limit lower=-2.3562 upper=0.6108 effort=50 velocity=35.2 -> lower=-2.3562 upper=0.6108 effort=61 velocity=35.2
- joint J20_SHOULDER_YAW_R: limit lower=-2.618 upper=2.618 effort=50 velocity=35.2 -> lower=-2.618 upper=2.618 effort=61 velocity=35.2
- joint J21_ELBOW_PITCH_R: limit lower=-2.1948 upper=0.7374 effort=50 velocity=35.2 -> lower=-2.1948 upper=0.7374 effort=61 velocity=35.2
- joint J22_ELBOW_YAW_R: limit lower=-2.618 upper=2.618 effort=50 velocity=35.2 -> lower=-2.618 upper=2.618 effort=61 velocity=35.2
- joint J23_HEAD_YAW: limit lower=-0.6109 upper=0.6109 effort=50 velocity=35.2 -> lower=-0.6109 upper=0.6109 effort=61 velocity=35.2
